File: pcb/bluetoothkiste.kicad_pcb (KiCad board)
At the start: 2 copper layers, 44.9 x 95.6 mm, 21 parts, among them J1 DB9_Female, J2 Screw_Terminal_01x03, J3 Screw_Terminal_01x03, J4 RJ45, J5 USB_A, J6 Conn_01x04_Female, J7 Screw_Terminal_01x03, U1 L7805, U2 MAX232

Commit message: beschriftungen pcb
Connections:
- J3 pad 1: /COMMON-TX -> /FLARM-TX
- J3 pad 2: /COMMON-RX -> /LX-TX
- J3 pad 3: /FLARM-TX -> /COMMON-TX
- J7 pad 1: /FLARM-RX -> /COMMON-RX
- J7 pad 2: /LX-TX -> /LX-RX
- J7 pad 3: /LX-RX -> /FLARM-RX
Other:
- board text added: "(Switched BAT+)"
- board text added: "Akaflieg Berlin Bluetoothkiste v1.0"
- board text added: "BAT+"
- board text added: "BAT-"
- board text added: "Common"
- board text added: "FLARM"
- board text added: "Fuse 2A"
- board text added: "GND"
- board text added: "HC-06"
- board text added: "LX"
- board text added: "PWR"
- board text added: "RX"
- board text added: "RXD"
- board text added: "TX"
- board text added: "TXD"
- board text added: "VCC"
Changed lines of the file:
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@@
   (general
     (thickness 1.6)
-    (drawings 16)
+    (drawings 32)
     (tracks 0)
     (zones 0)
@@
     (tags "mounting hole 3.2mm no annular m3")
     (attr virtual)
-    (fp_text reference REF** (at 0 -4.2) (layer F.SilkS)
+    (fp_text reference REF** (at 0 -4.2) (layer F.SilkS) hide
       (effects (font (size 1 1) (thickness 0.15)))
     )
@@
     (tags "mounting hole 3.2mm no annular m3")
     (attr virtual)
-    (fp_text reference REF** (at 0 -4.2) (layer F.SilkS)
+    (fp_text reference REF** (at 0 -4.2) (layer F.SilkS) hide
       (effects (font (size 1 1) (thickness 0.15)))
     )
@@
     (tags "mounting hole 3.2mm no annular m3")
     (attr virtual)
-    (fp_text reference REF** (at 0 -4.2) (layer F.SilkS)
+    (fp_text reference REF** (at 0 -4.2) (layer F.SilkS) hide
       (effects (font (size 1 1) (thickness 0.15)))
     )
@@
     (tags "mounting hole 3.2mm no annular m3")
     (attr virtual)
-    (fp_text reference REF** (at 0 -4.2) (layer F.SilkS)
+    (fp_text reference REF** (at 0 -4.2) (layer F.SilkS) hide
       (effects (font (size 1 1) (thickness 0.15)))
     )
@@
     (descr "Fuse, Fuseholder, TR5, Littelfuse/Wickmann, No. 460, No560, https://www.littelfuse.com/~/media/electronics/datasheets/fuse_holders/littelfuse_fuse_holder_559_560_datasheet.pdf.pdf")
     (tags "Fuse Fuseholder TR5 Littelfuse/Wickmann No. 460 No560 ")
-    (fp_text reference F1 (at 2.39 -6.89) (layer F.SilkS)
+    (fp_text reference F1 (at 2.8 -2.7) (layer F.SilkS)
       (effects (font (size 1 1) (thickness 0.15)))
     )
@@
     (descr "terminal block Metz Connect Type059_RT06303HBWC, 3 pins, pitch 3.5mm, size 10.5x6.5mm^2, drill diamater 1.2mm, pad diameter 2.3mm, see http://www.metz-connect.com/de/system/files/productfiles/Datenblatt_310591_RT063xxHBWC_OFF-022684T.pdf, script-generated using https://github.com/pointhi/kicad-footprint-generator/scripts/TerminalBlock_MetzConnect")
     (tags "THT terminal block Metz Connect Type059_RT06303HBWC pitch 3.5mm size 10.5x6.5mm^2 drill 1.2mm pad 2.3mm")
-    (fp_text reference J2 (at 3.5 -3.86 90) (layer F.SilkS)
+    (fp_text reference J2 (at 3.5 2.9 90) (layer F.SilkS)
       (effects (font (size 1 1) (thickness 0.15)))
     )
@@
       (effects (font (size 1 1) (thickness 0.15)))
     )
-    (fp_text value Screw_Terminal_01x03 (at 3.5 4.76) (layer F.Fab)
+    (fp_text value Screw_Terminal_01x03 (at 18.8 0.2) (layer F.Fab)
       (effects (font (size 1 1) (thickness 0.15)))
     )
@@
     (fp_arc (start 0 0) (end 0 1.555) (angle -27) (layer F.SilkS) (width 0.12))
     (pad 3 thru_hole circle (at 7 0) (size 2.3 2.3) (drill 1.2) (layers *.Cu *.Mask)
+      (net 14 /COMMON-TX))
+    (pad 2 thru_hole circle (at 3.5 0) (size 2.3 2.3) (drill 1.2) (layers *.Cu *.Mask)
+      (net 12 /LX-TX))
+    (pad 1 thru_hole rect (at 0 0) (size 2.3 2.3) (drill 1.2) (layers *.Cu *.Mask)
       (net 16 /FLARM-TX))
-    (pad 2 thru_hole circle (at 3.5 0) (size 2.3 2.3) (drill 1.2) (layers *.Cu *.Mask)
-      (net 15 /COMMON-RX))
-    (pad 1 thru_hole rect (at 0 0) (size 2.3 2.3) (drill 1.2) (layers *.Cu *.Mask)
-      (net 14 /COMMON-TX))
     (model ${KISYS3DMOD}/TerminalBlock_MetzConnect.3dshapes/TerminalBlock_MetzConnect_Type059_RT06303HBWC_1x03_P3.50mm_Horizontal.wrl
       (at (xyz 0 0 0))
@@
       (effects (font (size 1 1) (thickness 0.15)))
     )
-    (fp_text value Screw_Terminal_01x03 (at 3.5 4.76) (layer F.Fab)
+    (fp_text value Screw_Terminal_01x03 (at -12.1 0) (layer F.Fab)
       (effects (font (size 1 1) (thickness 0.15)))
     )
@@
     )
     (pad 1 thru_hole rect (at 0 0 180) (size 2.3 2.3) (drill 1.2) (layers *.Cu *.Mask)
+      (net 15 /COMMON-RX))
+    (pad 2 thru_hole circle (at 3.5 0 180) (size 2.3 2.3) (drill 1.2) (layers *.Cu *.Mask)
+      (net 11 /LX-RX))
+    (pad 3 thru_hole circle (at 7 0 180) (size 2.3 2.3) (drill 1.2) (layers *.Cu *.Mask)
       (net 17 /FLARM-RX))
-    (pad 2 thru_hole circle (at 3.5 0 180) (size 2.3 2.3) (drill 1.2) (layers *.Cu *.Mask)
-      (net 12 /LX-TX))
-    (pad 3 thru_hole circle (at 7 0 180) (size 2.3 2.3) (drill 1.2) (layers *.Cu *.Mask)
-      (net 11 /LX-RX))
     (model ${KISYS3DMOD}/TerminalBlock_MetzConnect.3dshapes/TerminalBlock_MetzConnect_Type059_RT06303HBWC_1x03_P3.50mm_Horizontal.wrl
       (at (xyz 0 0 0))
@@
     )
   )
+  (gr_text "(Switched BAT+)" (at 176.4 24.1) (layer F.SilkS)
+    (effects (font (size 0.7 0.7) (thickness 0.1)))
+  )
+  (gr_text RX (at 194.5 51.8) (layer F.SilkS)
+    (effects (font (size 1.5 1.5) (thickness 0.3)))
+  )
+  (gr_text TX (at 194.5 47) (layer F.SilkS)
+    (effects (font (size 1.5 1.5) (thickness 0.3)))
+  )
+  (gr_text FLARM (at 190.8 49.2) (layer F.SilkS)
+    (effects (font (size 0.8 0.8) (thickness 0.2)))
+  )
+  (gr_text LX (at 194.4 49.2) (layer F.SilkS)
+    (effects (font (size 0.8 0.8) (thickness 0.2)))
+  )
+  (gr_text Common (at 198.1 49.2) (layer F.SilkS)
+    (effects (font (size 0.8 0.8) (thickness 0.2)))
+  )
+  (gr_text "Fuse\n2A" (at 173 33) (layer F.SilkS)
+    (effects (font (size 1.5 1.5) (thickness 0.3)) (justify right))
+  )
+  (gr_text BAT+ (at 175.3 26.2) (layer F.SilkS)
+    (effects (font (size 1.5 1.5) (thickness 0.3)))
+  )
+  (gr_text PWR (at 174.764286 22.2) (layer F.SilkS)
+    (effects (font (size 1.5 1.5) (thickness 0.3)))
+  )
+  (gr_text BAT- (at 175.3 19.7) (layer F.SilkS)
+    (effects (font (size 1.5 1.5) (thickness 0.3)))
+  )
+  (gr_text GND (at 185 75.5 90) (layer F.SilkS)
+    (effects (font (size 1.5 1.5) (thickness 0.3)) (justify right))
+  )
+  (gr_text TXD (at 182.5 75.5 90) (layer F.SilkS)
+    (effects (font (size 1.5 1.5) (thickness 0.3)) (justify right))
+  )
+  (gr_text RXD (at 179.8 75.5 90) (layer F.SilkS)
+    (effects (font (size 1.5 1.5) (thickness 0.3)) (justify right))
+  )
+  (gr_text VCC (at 187.6 75.5 90) (layer F.SilkS)
+    (effects (font (size 1.5 1.5) (thickness 0.3)) (justify right))
+  )
+  (gr_text HC-06 (at 184.2 93.7) (layer F.SilkS)
+    (effects (font (size 1.5 1.5) (thickness 0.3)))
+  )
+  (gr_text "Akaflieg Berlin\nBluetoothkiste v1.0" (at 196.4 91.2 90) (layer F.SilkS)
+    (effects (font (size 2 2) (thickness 0.3)) (justify left))
+  )
   (gr_line (start 192.7 105) (end 192.7 112.5) (layer Edge.Cuts) (width 0.05))

Commit message: pcb layout
Parts:
- added G***: LOGO, footprints:Charlotte_5x5mm, F.Cu at (196.3, 94.9)
Routing:
- net +5V: track 0.00 -> 74.3 mm
- net /COMMON-RX: track 0.00 -> 72.7 mm, vias 0 -> 1
- net +12V: track 0.00 -> 70.1 mm, vias 0 -> 2
- net /FLARM-TX: track 0.00 -> 62.0 mm, vias 0 -> 1
- net /COMMON-TX: track 0.00 -> 52.5 mm, vias 0 -> 1
- net /LX-TX: track 0.00 -> 46.9 mm
- net /FLARM-RX: track 0.00 -> 42.3 mm, vias 0 -> 1
- net /LX-RX: track 0.00 -> 34.5 mm
- net Net-(C1-Pad1): track 0.00 -> 17.0 mm
- net /BT-RX: track 0.00 -> 16.5 mm
- net /BT-TX: track 0.00 -> 12.9 mm
- net +12P: track 0.00 -> 10.4 mm
- net Net-(C5-Pad2): track 0.00 -> 6.40 mm
- net Net-(C3-Pad1): track 0.00 -> 4.16 mm
- net Net-(C3-Pad2): track 0.00 -> 3.25 mm
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- added copper zone on B.Cu, net GND
- added copper zone on F.Cu, net GND

Commit message: vias
Parts:
- added REF**: VIA-0.6mm, JS_Local:VIA-0.6mm, F.Cu at (167.0, 101.0)
- added REF**: VIA-0.6mm, JS_Local:VIA-0.6mm, F.Cu at (160.0, 33.0)
- added REF**: VIA-0.6mm, JS_Local:VIA-0.6mm, F.Cu at (158.0, 33.0)
- added REF**: VIA-0.6mm, JS_Local:VIA-0.6mm, F.Cu at (165.0, 66.0)
- added REF**: VIA-0.6mm, JS_Local:VIA-0.6mm, F.Cu at (161.0, 68.0)
- added REF**: VIA-0.6mm, JS_Local:VIA-0.6mm, F.Cu at (159.0, 68.0)
- added REF**: VIA-0.6mm, JS_Local:VIA-0.6mm, F.Cu at (163.0, 66.0)
- added REF**: VIA-0.6mm, JS_Local:VIA-0.6mm, F.Cu at (161.0, 66.0)
- added REF**: VIA-0.6mm, JS_Local:VIA-0.6mm, F.Cu at (159.0, 66.0)
- added REF**: VIA-0.6mm, JS_Local:VIA-0.6mm, F.Cu at (198.0, 36.0)
- added REF**: VIA-0.6mm, JS_Local:VIA-0.6mm, F.Cu at (198.0, 34.0)
- added REF**: VIA-0.6mm, JS_Local:VIA-0.6mm, F.Cu at (169.0, 101.0)
- added REF**: VIA-0.6mm, JS_Local:VIA-0.6mm, F.Cu at (196.0, 36.0)
- added REF**: VIA-0.6mm, JS_Local:VIA-0.6mm, F.Cu at (196.0, 34.0)
- added REF**: VIA-0.6mm, JS_Local:VIA-0.6mm, F.Cu at (192.0, 36.0)
- added REF**: VIA-0.6mm, JS_Local:VIA-0.6mm, F.Cu at (194.0, 36.0)
- added REF**: VIA-0.6mm, JS_Local:VIA-0.6mm, F.Cu at (194.0, 34.0)
- added REF**: VIA-0.6mm, JS_Local:VIA-0.6mm, F.Cu at (192.0, 34.0)
- added REF**: VIA-0.6mm, JS_Local:VIA-0.6mm, F.Cu at (171.0, 101.0)
- added REF**: VIA-0.6mm, JS_Local:VIA-0.6mm, F.Cu at (173.0, 101.0)
- added REF**: VIA-0.6mm, JS_Local:VIA-0.6mm, F.Cu at (173.0, 99.0)
- added REF**: VIA-0.6mm, JS_Local:VIA-0.6mm, F.Cu at (171.0, 99.0)
- added REF**: VIA-0.6mm, JS_Local:VIA-0.6mm, F.Cu at (169.0, 99.0)
- added REF**: VIA-0.6mm, JS_Local:VIA-0.6mm, F.Cu at (167.0, 99.0)
- added REF**: VIA-0.6mm, JS_Local:VIA-0.6mm, F.Cu at (162.0, 33.0)

Commit message: dual channel
Parts:
- removed J5: USB_A, JS_Local:USB_A_UPRIGHT_SEGOR
- removed J7: Screw_Terminal_01x03, TerminalBlock_MetzConnect:TerminalBlock_MetzConnect_Type059_RT06303HBWC_1x03_P3.50mm_Horizontal
- removed the REF** at (165.0, 66.0)
- removed the REF** at (161.0, 68.0)
- removed the REF** at (159.0, 68.0)
- removed the REF** at (163.0, 66.0)
- removed the REF** at (161.0, 66.0)
- removed the REF** at (159.0, 66.0)
- removed the REF** at (198.0, 36.0)
- removed the REF** at (198.0, 34.0)
- removed the REF** at (196.0, 36.0)
- removed the REF** at (196.0, 34.0)
- removed the REF** at (192.0, 36.0)
- removed the REF** at (194.0, 36.0)
- removed the REF** at (194.0, 34.0)
- removed the REF** at (192.0, 34.0)
- added REF**: VIA-0.6mm, JS_Local:VIA-0.6mm, F.Cu at (187.0, 60.0)
- added REF**: VIA-0.6mm, JS_Local:VIA-0.6mm, F.Cu at (169.0, 74.0)
- added REF**: VIA-0.6mm, JS_Local:VIA-0.6mm, F.Cu at (164.0, 33.0)
- added REF**: VIA-0.6mm, JS_Local:VIA-0.6mm, F.Cu at (158.0, 37.0)
- added REF**: VIA-0.6mm, JS_Local:VIA-0.6mm, F.Cu at (158.0, 35.0)
- added REF**: VIA-0.6mm, JS_Local:VIA-0.6mm, F.Cu at (164.0, 35.0)
- added REF**: VIA-0.6mm, JS_Local:VIA-0.6mm, F.Cu at (162.0, 37.0)
- added REF**: VIA-0.6mm, JS_Local:VIA-0.6mm, F.Cu at (160.0, 35.0)
- added REF**: VIA-0.6mm, JS_Local:VIA-0.6mm, F.Cu at (160.0, 37.0)
- added REF**: VIA-0.6mm, JS_Local:VIA-0.6mm, F.Cu at (162.0, 35.0)
- added REF**: VIA-0.6mm, JS_Local:VIA-0.6mm, F.Cu at (164.0, 37.0)
- added REF**: VIA-0.6mm, JS_Local:VIA-0.6mm, F.Cu at (191.0, 60.0)
- added REF**: VIA-0.6mm, JS_Local:VIA-0.6mm, F.Cu at (161.0, 74.0)
- added REF**: VIA-0.6mm, JS_Local:VIA-0.6mm, F.Cu at (161.0, 72.0)
- added REF**: VIA-0.6mm, JS_Local:VIA-0.6mm, F.Cu at (163.0, 72.0)
- added REF**: VIA-0.6mm, JS_Local:VIA-0.6mm, F.Cu at (165.0, 72.0)
- added REF**: VIA-0.6mm, JS_Local:VIA-0.6mm, F.Cu at (165.0, 74.0)
- added REF**: VIA-0.6mm, JS_Local:VIA-0.6mm, F.Cu at (163.0, 74.0)
- added REF**: VIA-0.6mm, JS_Local:VIA-0.6mm, F.Cu at (159.0, 72.0)
- added REF**: VIA-0.6mm, JS_Local:VIA-0.6mm, F.Cu at (159.0, 74.0)
- added REF**: VIA-0.6mm, JS_Local:VIA-0.6mm, F.Cu at (195.0, 60.0)
- added REF**: VIA-0.6mm, JS_Local:VIA-0.6mm, F.Cu at (197.0, 60.0)
- added REF**: VIA-0.6mm, JS_Local:VIA-0.6mm, F.Cu at (189.0, 60.0)
- added REF**: VIA-0.6mm, JS_Local:VIA-0.6mm, F.Cu at (193.0, 60.0)
- added REF**: VIA-0.6mm, JS_Local:VIA-0.6mm, F.Cu at (169.0, 72.0)
- added REF**: VIA-0.6mm, JS_Local:VIA-0.6mm, F.Cu at (167.0, 74.0)
- added REF**: VIA-0.6mm, JS_Local:VIA-0.6mm, F.Cu at (167.0, 72.0)
- J3: value Screw_Terminal_01x03 -> Conn_01x04_Female; footprint TerminalBlock_MetzConnect:TerminalBlock_MetzConnect_Type059_RT06303HBWC_1x03_P3.50mm_Horizontal -> Connector_PinSocket_2.54mm:PinSocket_1x04_P2.54mm_Horizontal
- moved J3 6.03 mm to (187.7, 35.8), turned to 90 degrees
- moved C7 5.55 mm to (181.5, 38.9)
- moved J1 5.00 mm to (164.6, 60.0)
- moved C3 3.46 mm to (172.3, 45.0)
- moved C4 3.46 mm to (172.3, 51.0)
- moved C5 3.46 mm to (169.3, 43.0)
- moved C6 3.46 mm to (170.7, 55.0)
- moved U2 3.46 mm to (175.3, 42.0)
- moved J4 1.88 mm to (168.8, 82.0)
- moved C1 1.22 mm to (187.0, 29.0)
- moved U1 0.80 mm to (183.6, 25.0)
- moved C2 0.70 mm to (191.9, 32.0)
Connections:
- J3 pad 1: /FLARM-TX -> /LX-BT-RX
- J3 pad 2: /LX-TX -> /LX-BT-TX
- J3 pad 3: /COMMON-TX -> GND
- J6 pad 1: /BT-RX -> /FLARM-BT-RX
- J6 pad 2: /BT-TX -> /FLARM-BT-TX
- U2 pad 10: (no net) -> /FLARM-BT-TX
- U2 pad 11: /BT-TX -> /LX-BT-TX
- U2 pad 12: /BT-RX -> /LX-BT-RX
- U2 pad 13: /COMMON-TX -> /LX-TX
- U2 pad 14: /COMMON-RX -> /LX-RX
- U2 pad 7: (no net) -> /FLARM-RX
- U2 pad 8: (no net) -> /FLARM-TX
- U2 pad 9: (no net) -> /FLARM-BT-RX
Routing:
- net /COMMON-RX: track 72.7 -> 0.00 mm, vias 1 -> 0
- net /COMMON-TX: track 52.5 -> 0.00 mm, vias 1 -> 0
- net /FLARM-TX: track 62.0 -> 30.8 mm, vias 1 -> 2
- net /LX-BT-TX: track 0.00 -> 22.0 mm
- net /LX-BT-RX: track 0.00 -> 18.4 mm
- net +5V: track 74.3 -> 56.9 mm
- net /BT-RX: track 16.5 -> 0.00 mm
- net /LX-TX: track 46.9 -> 33.9 mm, vias 0 -> 1
- net /BT-TX: track 12.9 -> 0.00 mm
- net /FLARM-BT-TX: track 0.00 -> 8.75 mm
- net /FLARM-RX: track 42.3 -> 33.7 mm, vias 1 -> 0
- net Net-(C1-Pad1): track 17.0 -> 11.3 mm
- net /FLARM-BT-RX: track 0.00 -> 5.34 mm
- net +12V: track 70.1 -> 65.9 mm, vias 2 -> 0
- net /LX-RX: track 34.5 -> 31.1 mm, vias 0 -> 1
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Other:
- board text added: "HC-06 FLARM"
- board text added: "HC-06 LX"
- board text removed: "Common"
- board text removed: "FLARM"
- board text removed: "HC-06"
- board text removed: "LX"
- board text removed: "RX"
- board text removed: "TX"
